File: PiPan-Keyboard.kicad_sch (KiCad schematic)
At the start: 149 parts, among them J0 Conn_01x18_MountingPin, SW0 RotaryEncoder_Switch, U1 Pico

Commit message: placed diodes
Parts:
- renumbered D41 to D10, D5 to D11, D45 to D12, D6 to D13, D10 to D14, D14 to D15, D18 to D16, D22 to D17, D26 to D18, D30 to D19, D9 to D2, D34 to D20, D38 to D21, D42 to D22, D3 to D23, D7 to D24, D11 to D25, D15 to D26, D19 to D27, D23 to D28, D27 to D29, D13 to D3, D31 to D30, D35 to D31, D39 to D32, D43 to D33, D4 to D34, D8 to D35, D12 to D36, D16 to D37, D20 to D38, D24 to D39, D17 to D4, D28 to D40, D32 to D41, D36 to D42, D40 to D43, D46 to D45, D47 to D46, D48 to D47, D49 to D48, D21 to D5, D25 to D6, D29 to D7, D33 to D8, D37 to D9
Connections:
- net at D27.2 (A): now also MX26.2 (ROW)
- net at D16.2 (A): now also MX15.2 (ROW)
- net at D40.2 (A): now also MX39.2 (ROW)
- net at D28.2 (A): now also MX27.2 (ROW)
- net at MX38.2 (ROW): now also D39.2 (A)
- net at MX37.2 (ROW): now also D38.2 (A)

Commit message: added outline to kaihl mx footprint andfixedlayout
Parts:
- MX0, MX1, MX10, MX11, MX12, MX13, MX14, MX15, MX16, MX17, MX18, MX19, MX2, MX20, MX21, MX22, MX23, MX24, MX25, MX26, MX27, MX28, MX29, MX3, MX30, MX31, MX32, MX33, MX34, MX35, MX36, MX37, MX38, MX39, MX4, MX40, MX41, MX42, MX43, MX44, MX45, MX46, MX47, MX5, MX6, MX7, MX8, MX9: footprint keyswitches:Kailh_socket_MX -> keyswitches:Kailh_socket_MX-Outlined
