File: PiPan-Keyboard.kicad_pcb (KiCad board)
At the start: 2 copper layers, 93 parts, among them J0 Conn_01x18_MountingPin, SW0 RotaryEncoder_Switch, U1 Pico

Commit message: placed first row
Parts:
- moved D1 305.6 mm to (566.9, 201.7)
- moved D16 305.6 mm to (590.7, 209.7)
- moved D25 305.6 mm to (590.7, 206.1)
- moved D7 305.6 mm to (567.7, 224.6)
- moved D8 305.6 mm to (567.7, 221.1)
- moved D12 305.6 mm to (583.9, 199.3)
- moved D23 305.6 mm to (583.9, 195.8)
- moved D28 305.6 mm to (583.9, 192.2)
- moved D3 305.6 mm to (577.4, 206.1)
- moved D33 305.6 mm to (567.7, 195.4)
- moved D35 305.6 mm to (579.6, 216.0)
- moved D37 305.6 mm to (581.0, 221.1)
- moved D38 305.6 mm to (581.0, 224.6)
- moved D4 305.6 mm to (567.7, 191.8)
- moved D17 279.5 mm to (559.7, 168.9)
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
Commit message: corrected switches in schema
Parts:
- moved MX26 471.1 mm to (110.3, 93.7)
- moved MX28 421.0 mm to (140.5, 93.7)
- moved MX18 410.7 mm to (170.7, 78.6)
- moved MX29 405.4 mm to (155.6, 93.7)
- moved MX15 374.1 mm to (125.4, 78.6)
- moved MX14 367.9 mm to (110.3, 78.6)
- moved MX25 367.2 mm to (95.2, 93.7)
- moved MX24 359.3 mm to (80.2, 93.7)
- moved MX19 356.9 mm to (185.7, 78.6)
- moved MX27 332.4 mm to (125.4, 93.7)
- moved MX33 289.6 mm to (215.9, 93.7)
- moved MX22 287.7 mm to (231.0, 78.6)
- moved MX20 282.0 mm to (200.8, 78.6)
- moved MX16 281.7 mm to (140.5, 78.6)
- moved MX31 279.5 mm to (185.7, 93.7)
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Changed lines of the file:
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@@
   (net 87 "COL11")
   (footprint "keyswitches:Kailh_socket_MX" (layer "F.Cu")
-    (at 437.62 150.58875)
+    (at 200.81875 93.6625)
     (descr "MX-style keyswitch with Kailh socket mount")
     (tags "MX,cherry,gateron,kailh,pg1511,socket")
@@
   )
   (footprint "keyswitches:Kailh_socket_MX" (layer "F.Cu")
-    (at 560.92625 71.37625)
+    (at 140.49375 93.6625)
     (descr "MX-style keyswitch with Kailh socket mount")
     (tags "MX,cherry,gateron,kailh,pg1511,socket")
@@
   )
   (footprint "keyswitches:Kailh_socket_MX" (layer "F.Cu")
-    (at 498.22 110.18875)
+    (at 125.4125 78.58125)
     (descr "MX-style keyswitch with Kailh socket mount")
     (tags "MX,cherry,gateron,kailh,pg1511,socket")
@@
   )
   (footprint "keyswitches:Kailh_socket_MX" (layer "F.Cu")
-    (at 478.02 130.38875)
+    (at 200.81875 78.58125)
     (descr "MX-style keyswitch with Kailh socket mount")
     (tags "MX,cherry,gateron,kailh,pg1511,socket")
@@
   )
   (footprint "keyswitches:Kailh_socket_MX" (layer "F.Cu")
-    (at 542.5 69.78875)
+    (at 185.7375 78.58125)
     (descr "MX-style keyswitch with Kailh socket mount")
     (tags "MX,cherry,gateron,kailh,pg1511,socket")
@@
   )
   (footprint "keyswitches:Kailh_socket_MX" (layer "F.Cu")
-    (at 478.02 89.98875)
+    (at 110.33125 78.58125)
     (descr "MX-style keyswitch with Kailh socket mount")
     (tags "MX,cherry,gateron,kailh,pg1511,socket")
@@
   )
   (footprint "keyswitches:Kailh_socket_MX" (layer "F.Cu")
-    (at 421.3 69.78875)
+    (at 215.9 78.58125)
     (descr "MX-style keyswitch with Kailh socket mount")
     (tags "MX,cherry,gateron,kailh,pg1511,socket")
@@
   )
   (footprint "keyswitches:Kailh_socket_MX" (layer "F.Cu")
-    (at 457.82 89.98875)
+    (at 125.4125 93.6625)
     (descr "MX-style keyswitch with Kailh socket mount")
     (tags "MX,cherry,gateron,kailh,pg1511,socket")
@@
   )
   (footprint "keyswitches:Kailh_socket_MX" (layer "F.Cu")
-    (at 502.1 49.58875)
+    (at 215.9 93.6625)
     (descr "MX-style keyswitch with Kailh socket mount")
     (tags "MX,cherry,gateron,kailh,pg1511,socket")
@@
   )
   (footprint "keyswitches:Kailh_socket_MX" (layer "F.Cu")
-    (at 581.12625 91.57625)
+    (at 170.65625 78.58125)
     (descr "MX-style keyswitch with Kailh socket mount")
     (tags "MX,cherry,gateron,kailh,pg1511,socket")
@@
   )
   (footprint "keyswitches:Kailh_socket_MX" (layer "F.Cu")
-    (at 461.7 69.78875)
+    (at 95.25 93.6625)
     (descr "MX-style keyswitch with Kailh socket mount")
     (tags "MX,cherry,gateron,kailh,pg1511,socket")
@@
   )
   (footprint "keyswitches:Kailh_socket_MX" (layer "F.Cu")
-    (at 401.1 49.58875)
+    (at 155.575 78.58125)
     (descr "MX-style keyswitch with Kailh socket mount")
     (tags "MX,cherry,gateron,kailh,pg1511,socket")
@@
   )
   (footprint "keyswitches:Kailh_socket_MX" (layer "F.Cu")
-    (at 417.42 130.38875)
+    (at 140.49375 78.58125)
     (descr "MX-style keyswitch with Kailh socket mount")
     (tags "MX,cherry,gateron,kailh,pg1511,socket")
@@
   )
   (footprint "keyswitches:Kailh_socket_MX" (layer "F.Cu")
-    (at 461.7 49.58875)
+    (at 185.7375 93.6625)
     (descr "MX-style keyswitch with Kailh socket mount")
     (tags "MX,cherry,gateron,kailh,pg1511,socket")
@@
   )
   (footprint "keyswitches:Kailh_socket_MX" (layer "F.Cu")
-    (at 518.42 89.98875)
+    (at 230.98125 78.58125)
     (descr "MX-style keyswitch with Kailh socket mount")
     (tags "MX,cherry,gateron,kailh,pg1511,socket")
@@
   )
   (footprint "keyswitches:Kailh_socket_MX" (layer "F.Cu")
-    (at 457.82 150.58875)
+    (at 246.0625 78.58125)
     (descr "MX-style keyswitch with Kailh socket mount")
     (tags "MX,cherry,gateron,kailh,pg1511,socket")
@@
   )
   (footprint "keyswitches:Kailh_socket_MX" (layer "F.Cu")
-    (at 417.42 110.18875)
+    (at 170.65625 93.6625)
     (descr "MX-style keyswitch with Kailh socket mount")
     (tags "MX,cherry,gateron,kailh,pg1511,socket")
@@
   )
   (footprint "keyswitches:Kailh_socket_MX" (layer "F.Cu")
-    (at 437.62 130.38875)
+    (at 80.16875 93.6625)
     (descr "MX-style keyswitch with Kailh socket mount")
     (tags "MX,cherry,gateron,kailh,pg1511,socket")
@@
   )
   (footprint "keyswitches:Kailh_socket_MX" (layer "F.Cu")
-    (at 581.12625 111.77625)
+    (at 110.33125 93.6625)
     (descr "MX-style keyswitch with Kailh socket mount")
     (tags "MX,cherry,gateron,kailh,pg1511,socket")
@@
   )
   (footprint "keyswitches:Kailh_socket_MX" (layer "F.Cu")
-    (at 481.9 69.78875)
+    (at 230.98125 93.6625)
     (descr "MX-style keyswitch with Kailh socket mount")
     (tags "MX,cherry,gateron,kailh,pg1511,socket")
@@
   )
   (footprint "keyswitches:Kailh_socket_MX" (layer "F.Cu")
-    (at 560.92625 91.57625)
+    (at 155.575 93.6625)
     (descr "MX-style keyswitch with Kailh socket mount")
     (tags "MX,cherry,gateron,kailh,pg1511,socket")

Commit message: updated PCB with added components
Parts:
- added D46: D_Small, Diode_THT:D_DO-35_SOD27_P10.16mm_Horizontal, F.Cu at (442.1, 140.5)
- added D47: D_Small, Diode_THT:D_DO-35_SOD27_P10.16mm_Horizontal, F.Cu at (442.1, 144.0)
- added D48: D_Small, Diode_THT:D_DO-35_SOD27_P10.16mm_Horizontal, F.Cu at (442.1, 133.4)
- added D49: D_Small, Diode_THT:D_DO-35_SOD27_P10.16mm_Horizontal, F.Cu at (442.1, 136.9)
- added MX44: MX-NoLED, keyswitches:Kailh_socket_MX, F.Cu at (432.4, 139.7)
- added MX45: MX-NoLED, keyswitches:Kailh_socket_MX, F.Cu at (432.4, 155.8)
- added MX46: MX-NoLED, keyswitches:Kailh_socket_MX, F.Cu at (414.7, 155.8)
- added MX47: MX-NoLED, keyswitches:Kailh_socket_MX, F.Cu at (414.7, 139.7)
Connections:
- D12 pad 1: ROW3 -> ROW2
- D18 pad 2: Net-(D18-Pad2) -> unconnected-(D18-Pad2)
- D19 pad 2: Net-(D19-Pad2) -> unconnected-(D19-Pad2)
- D2 pad 1: ROW1 -> ROW0
- D20 pad 2: Net-(D20-Pad2) -> unconnected-(D20-Pad2)
- D23 pad 2: Net-(D23-Pad2) -> unconnected-(D23-Pad2)
- D24 pad 2: Net-(D24-Pad2) -> unconnected-(D24-Pad2)
- D28 pad 2: Net-(D28-Pad2) -> unconnected-(D28-Pad2)
- D3 pad 1: ROW2 -> ROW1
- D4 pad 1: ROW3 -> ROW2
- D7 pad 1: ROW2 -> ROW1
- D8 pad 1: ROW3 -> ROW2
- MX11 pad 1: COL0 -> COL11
- MX12 pad 1: COL1 -> COL0
- MX13 pad 1: COL2 -> COL1
- MX14 pad 1: COL3 -> COL2
- MX15 pad 1: COL4 -> unconnected-(MX15-Pad1)
- MX15 pad 2: Net-(D18-Pad2) -> unconnected-(MX15-Pad2)
- MX16 pad 1: COL5 -> COL4
- MX17 pad 1: COL6 -> COL5
- MX18 pad 1: COL7 -> COL6
- MX19 pad 1: COL8 -> COL7
- MX20 pad 1: COL9 -> COL8
- MX21 pad 1: COL10 -> COL9
- MX22 pad 1: COL0 -> COL10
- MX23 pad 1: COL1 -> COL11
- MX24 pad 1: COL2 -> COL0
- MX25 pad 1: COL3 -> COL1
- MX26 pad 1: COL4 -> unconnected-(MX26-Pad1)
- MX26 pad 2: Net-(D19-Pad2) -> unconnected-(MX26-Pad2)
- MX27 pad 1: COL5 -> unconnected-(MX27-Pad1)
- MX27 pad 2: Net-(D23-Pad2) -> unconnected-(MX27-Pad2)
- MX28 pad 1: COL6 -> COL4
- MX29 pad 1: COL7 -> COL5
- MX30 pad 1: COL8 -> COL6
- MX31 pad 1: COL9 -> COL7
- MX32 pad 1: COL10 -> COL8
- MX33 pad 1: COL0 -> COL9
- MX34 pad 1: COL1 -> COL10
- MX35 pad 1: COL2 -> COL11
- MX36 pad 1: COL3 -> COL0
- MX37 pad 1: COL4 -> unconnected-(MX37-Pad1)
- MX37 pad 2: Net-(D20-Pad2) -> unconnected-(MX37-Pad2)
- MX38 pad 1: COL5 -> unconnected-(MX38-Pad1)
- MX38 pad 2: Net-(D24-Pad2) -> unconnected-(MX38-Pad2)
- MX39 pad 1: COL6 -> unconnected-(MX39-Pad1)
- MX39 pad 2: Net-(D28-Pad2) -> unconnected-(MX39-Pad2)
- MX40 pad 1: COL7 -> COL4
- MX41 pad 1: COL8 -> COL5
- MX42 pad 1: COL9 -> COL6
- MX43 pad 1: COL10 -> COL7
- SW0 pad S2: COL11 -> COL12

Commit message: fixing diode labels in progress.
Parts:
- moved D1 510.2 mm to (74.3, 69.1)
- moved MX37 465.7 mm to (95.2, 108.7)
- moved MX39 421.5 mm to (125.4, 108.7)
- moved MX36 397.9 mm to (80.2, 108.7)
- moved D2 387.1 mm to (183.8, 40.5)
- moved MX38 376.2 mm to (110.3, 108.7)
- moved MX41 348.7 mm to (155.6, 108.7)
- moved MX42 347.8 mm to (170.7, 108.7)
- moved MX40 340.1 mm to (140.5, 108.7)
- moved MX43 313.0 mm to (185.7, 108.7)
- moved MX35 277.3 mm to (246.1, 93.7)
- moved MX44 233.6 mm to (200.8, 108.7)
- moved MX45 221.5 mm to (215.9, 108.7)
- moved MX46 189.7 mm to (231.0, 108.7)
- moved MX47 171.5 mm to (246.1, 108.7)
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
Commit message: placed diodes
Parts:
- D0: renamed from D1; moved to B.Cu
- D1: renamed from D2; moved to B.Cu
- D10: renamed from D41; moved to B.Cu
- D11: renamed from D5; moved to B.Cu
- D12: renamed from D45; moved to B.Cu
- D13: renamed from D6; moved to B.Cu
- D14: renamed from D10; moved to B.Cu
- D15: renamed from D14; moved to B.Cu
- D16: renamed from D18; moved to B.Cu
- D17: renamed from D22; moved to B.Cu
- D18: renamed from D26; moved to B.Cu
- D19: renamed from D30; moved to B.Cu
- D2: renamed from D9; moved to B.Cu
- D20: renamed from D34; moved to B.Cu
- D21: renamed from D38; moved to B.Cu
- D22: renamed from D42; moved to B.Cu
- D23: renamed from D3; moved to B.Cu
- D24: renamed from D7; moved to B.Cu
- D25: renamed from D11; moved to B.Cu
- D26: renamed from D15; moved to B.Cu
- D27: renamed from D19; moved to B.Cu
- D28: renamed from D23; moved to B.Cu
- D29: renamed from D27; moved to B.Cu
- D3: renamed from D13; moved to B.Cu
- D30: renamed from D31; moved to B.Cu
- D31: renamed from D35; moved to B.Cu
- D32: renamed from D39; moved to B.Cu
- D33: renamed from D43; moved to B.Cu
- D34: renamed from D4; moved to B.Cu
- D35: renamed from D8; moved to B.Cu
- D36: renamed from D12; moved to B.Cu
- D37: renamed from D16; moved to B.Cu
- D38: renamed from D20; moved to B.Cu
- D39: renamed from D24; moved to B.Cu
- D4: renamed from D17; moved to B.Cu
- D40: renamed from D28; moved to B.Cu
- D41: renamed from D32; moved to B.Cu
- D42: renamed from D36; moved to B.Cu
- D43: renamed from D40; moved to B.Cu
- D44: moved to B.Cu
- D45: renamed from D46; moved to B.Cu
- D46: renamed from D47; moved to B.Cu
- D47: renamed from D48; moved to B.Cu
- D48: renamed from D49; moved to B.Cu
- D5: renamed from D21; moved to B.Cu
- D6: renamed from D25; moved to B.Cu
- D7: renamed from D29; moved to B.Cu
- D8: renamed from D33; moved to B.Cu
- D9: renamed from D37; moved to B.Cu
- moved D12 526.0 mm to (49.5, 126.2), turned to 180 degrees
- moved D28 497.2 mm to (108.4, 106.4)
- moved D40 493.8 mm to (108.4, 121.4)
- moved D14 488.6 mm to (78.3, 91.3)
- moved D15 486.8 mm to (93.3, 91.3)
- moved D27 469.2 mm to (93.3, 106.4)
- moved D6 456.0 mm to (153.7, 76.2)
- moved D17 454.5 mm to (123.5, 91.3)
- moved D13 450.9 mm to (63.2, 91.3)
- moved D26 450.2 mm to (78.3, 106.4)
- moved D41 449.6 mm to (123.5, 121.4)
- moved D37 448.6 mm to (63.2, 121.4)
- moved D25 446.9 mm to (63.2, 106.4)
- moved D31 439.8 mm to (153.7, 106.4)
- moved D4 429.3 mm to (123.5, 76.2)
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Connections:
- D1 pad 2: Net-(D2-Pad2) (its old number) -> Net-(D1-Pad2)
- D11 pad 2: Net-(D5-Pad2) (its old number) -> Net-(D11-Pad2)
- D16 pad 2: unconnected-(D18-Pad2) -> Net-(D16-Pad2)
- D27 pad 2: unconnected-(D19-Pad2) -> Net-(MX26-Pad2)
- D28 pad 2: unconnected-(D23-Pad2) -> Net-(MX27-Pad2)
- D38 pad 2: unconnected-(D20-Pad2) -> Net-(D38-Pad2)
- D39 pad 2: unconnected-(D24-Pad2) -> Net-(MX38-Pad2)
- D40 pad 2: unconnected-(D28-Pad2) -> Net-(MX39-Pad2)
- MX1 pad 2: Net-(D5-Pad2) (its old number) -> Net-(D1-Pad2)
- MX11 pad 2: Net-(D2-Pad2) (its old number) -> Net-(D11-Pad2)
- MX15 pad 2: unconnected-(MX15-Pad2) -> Net-(D16-Pad2)
- MX26 pad 2: unconnected-(MX26-Pad2) -> Net-(MX26-Pad2)
- MX27 pad 2: unconnected-(MX27-Pad2) -> Net-(MX27-Pad2)
- MX37 pad 2: unconnected-(MX37-Pad2) -> Net-(D38-Pad2)
- MX38 pad 2: unconnected-(MX38-Pad2) -> Net-(MX38-Pad2)
- MX39 pad 2: unconnected-(MX39-Pad2) -> Net-(MX39-Pad2)

Commit message: generated first test step file
Parts:
- moved SW0 65.9 mm to (-21.5, 119.7), turned to 0 degrees
- moved D12 59.3 mm to (-9.21, 134.1)
- moved U1 0.79 mm to (44.5, 88.9)
- moved OL1 0.38 mm to (48.4, 118.3)
Other:
- board outline added: 216.7 x 61.1 mm
Changed lines of the file:
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@@
   )
   (footprint "Connector_PinSocket_2.54mm:PinSocket_1x04_P2.54mm_Horizontal" (layer "F.Cu")
-    (at 48.3 117.90625 -90)
+    (at 48.41875 118.26875 -90)
     (descr "Through hole angled socket strip, 1x04, 2.54mm pitch, 8.51mm socket length, single row (from Kicad 4.0.7), script generated")
     (tags "Through hole angled socket strip THT 1x04 2.54mm single row")
@@
   )
   (footprint "Rotary_Encoder:RotaryEncoder_Alps_EC11E-Switch_Vertical_H20mm" (layer "F.Cu")
-    (at 41.95 137.425 90)
+    (at -21.5375 119.7375)
     (descr "Alps rotary encoder, EC12E... with switch, vertical shaft, http://www.alps.com/prod/info/E/HTML/Encoder/Incremental/EC11/EC11E15204A3.html")
     (tags "rotary encoder")
@@
     (property "Sheetname" "")
     (attr through_hole)
-    (fp_text reference "SW0" (at 2.8 -4.7 90) (layer "F.SilkS")
+    (fp_text reference "SW0" (at 2.8 -4.7) (layer "F.SilkS")
       (effects (font (size 1 1) (thickness 0.15)))
     )
-    (fp_text value "RotaryEncoder_Switch" (at 7.5 10.4 90) (layer "F.Fab")
+    (fp_text value "RotaryEncoder_Switch" (at 7.5 10.4) (layer "F.Fab")
       (effects (font (size 1 1) (thickness 0.15)))
     )
-    (fp_text user "${REFERENCE}" (at 11.1 6.3 90) (layer "F.Fab")
+    (fp_text user "${REFERENCE}" (at 11.1 6.3) (layer "F.Fab")
       (effects (font (size 1 1) (thickness 0.15)))
     )
@@
     (fp_line (start 4.5 2.5) (end 10.5 2.5) (layer "F.Fab") (width 0.12))
     (fp_circle (center 7.5 2.5) (end 10.5 2.5) (layer "F.Fab") (width 0.12) (fill none))
-    (pad "A" thru_hole rect locked (at 0 0 90) (size 2 2) (drill 1) (layers *.Cu *.Mask)
+    (pad "A" thru_hole rect locked (at 0 0) (size 2 2) (drill 1) (layers *.Cu *.Mask)
       (net 19 "Encoder_A") (pinfunction "A") (pintype "passive"))
-    (pad "B" thru_hole circle locked (at 0 5 90) (size 2 2) (drill 1) (layers *.Cu *.Mask)
+    (pad "B" thru_hole circle locked (at 0 5) (size 2 2) (drill 1) (layers *.Cu *.Mask)
       (net 17 "Encoder_B") (pinfunction "B") (pintype "passive"))
-    (pad "C" thru_hole circle locked (at 0 2.5 90) (size 2 2) (drill 1) (layers *.Cu *.Mask)
+    (pad "C" thru_hole circle locked (at 0 2.5) (size 2 2) (drill 1) (layers *.Cu *.Mask)
       (net 22 "GND") (pinfunction "C") (pintype "passive"))
-    (pad "MP" thru_hole rect locked (at 7.5 -3.1 90) (size 3.2 2) (drill oval 2.8 1.5) (layers *.Cu *.Mask))
-    (pad "MP" thru_hole rect locked (at 7.5 8.1 90) (size 3.2 2) (drill oval 2.8 1.5) (layers *.Cu *.Mask))
-    (pad "S1" thru_hole circle locked (at 14.5 5 90) (size 2 2) (drill 1) (layers *.Cu *.Mask)
+    (pad "MP" thru_hole rect locked (at 7.5 -3.1) (size 3.2 2) (drill oval 2.8 1.5) (layers *.Cu *.Mask))
+    (pad "MP" thru_hole rect locked (at 7.5 8.1) (size 3.2 2) (drill oval 2.8 1.5) (layers *.Cu *.Mask))
+    (pad "S1" thru_hole circle locked (at 14.5 5) (size 2 2) (drill 1) (layers *.Cu *.Mask)
       (net 45 "Net-(D12-Pad2)") (pinfunction "S1") (pintype "passive"))
-    (pad "S2" thru_hole circle locked (at 14.5 0 90) (size 2 2) (drill 1) (layers *.Cu *.Mask)
+    (pad "S2" thru_hole circle locked (at 14.5 0) (size 2 2) (drill 1) (layers *.Cu *.Mask)
       (net 98 "COL12") (pinfunction "S2") (pintype "passive"))
     (model "${KISYS3DMOD}/Rotary_Encoder.3dshapes/RotaryEncoder_Alps_EC11E-Switch_Vertical_H20mm.wrl"
@@
   )
   (footprint "MCU_RaspberryPi_and_Boards:RPi_Pico_SMD_TH" (layer "F.Cu")
-    (at 44.45 89.69375)
+    (at 44.45 88.9)
     (descr "Through hole straight pin header, 2x20, 2.54mm pitch, double rows")
     (tags "Through hole pin header THT 2x20 2.54mm double row")
@@
   )
   (footprint "Diode_THT:D_DO-35_SOD27_P10.16mm_Horizontal" (layer "B.Cu")
-    (at 49.53 126.20625 180)
+    (at -9.2075 134.14375 180)
     (descr "Diode, DO-35_SOD27 series, Axial, Horizontal, pin pitch=10.16mm, , length*diameter=4*2mm^2, , http://www.diodes.com/_files/packages/DO-35.pdf")
     (tags "Diode DO-35_SOD27 series Axial Horizontal pin pitch 10.16mm  length 4mm diameter 2mm")
@@
     )
   )
+  (gr_arc (start 26.19375 123.825) (mid 25.632484 123.592516) (end 25.4 123.03125) (layer "Edge.Cuts") (width 0.1))
+  (gr_arc (start 25.4 63.5) (mid 25.632484 62.938734) (end 26.19375 62.70625) (layer "Edge.Cuts") (width 0.1))
+  (gr_line (start 26.19375 123.825) (end 241.3 123.825) (layer "Edge.Cuts") (width 0.1))
+  (gr_line (start 241.3 62.70625) (end 26.19375 62.70625) (layer "Edge.Cuts") (width 0.1))
+  (gr_arc (start 241.3 62.70625) (mid 241.861266 62.938734) (end 242.09375 63.5) (layer "Edge.Cuts") (width 0.1))
+  (gr_line (start 242.09375 123.03125) (end 242.09375 63.5) (layer "Edge.Cuts") (width 0.1))
+  (gr_line (start 25.4 63.5) (end 25.4 123.03125) (layer "Edge.Cuts") (width 0.1))
+  (gr_arc (start 242.09375 123.03125) (mid 241.861266 123.592516) (end 241.3 123.825) (layer "Edge.Cuts") (width 0.1))
 )

Commit message: added outline to kaihl mx footprint andfixedlayout
Parts:
- MX0, MX1, MX10, MX11, MX12, MX13, MX14, MX15, MX16, MX17, MX18, MX19, MX2, MX20, MX21, MX22, MX23, MX24, MX25, MX26, MX27, MX28, MX29, MX3, MX30, MX31, MX32, MX33, MX34, MX35, MX36, MX37, MX38, MX39, MX4, MX40, MX41, MX42, MX43, MX44, MX45, MX46, MX47, MX5, MX6, MX7, MX8, MX9: footprint keyswitches:Kailh_socket_MX -> keyswitches:Kailh_socket_MX-Outlined
- moved D12 65.6 mm to (55.6, 123.5), turned to -90 degrees
- moved SW0 59.1 mm to (37.2, 126.1)
- moved D48 45.3 mm to (272.7, 133.3)
- moved MX47 45.3 mm to (277.8, 127.8)
- moved D36 44.4 mm to (272.7, 114.3)
- moved MX35 44.4 mm to (277.8, 108.7)
- moved D24 43.8 mm to (272.7, 95.2)
- moved MX23 43.8 mm to (277.8, 89.7)
- moved D11 43.7 mm to (272.7, 76.2)
- moved MX11 43.7 mm to (277.8, 70.6)
- moved D47 41.4 mm to (253.7, 133.3)
- moved MX46 41.4 mm to (258.8, 127.8)
- moved D35 40.5 mm to (253.7, 114.3)
- moved MX34 40.5 mm to (258.8, 108.7)
- moved D23 39.9 mm to (253.7, 95.2)
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Other:
- board size 216.7 x 61.1 mm -> 262.7 x 76.2 mm

Commit message: adjusted board size and pico position
Parts:
- moved J0 1.69 mm to (29.4, 72.9)
- moved U1 1.59 mm to (44.5, 87.3)
- moved SW0 0.41 mm to (37.6, 126.1)
Other:
- board size 262.7 x 76.2 mm -> 260.3 x 76.2 mm
Changed lines of the file:
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@@
   )
   (footprint "Rotary_Encoder:RotaryEncoder_Alps_EC11E-Switch_Vertical_H20mm" (layer "F.Cu")
-    (at 37.2 126.0875)
+    (at 37.6125 126.0875)
     (descr "Alps rotary encoder, EC12E... with switch, vertical shaft, http://www.alps.com/prod/info/E/HTML/Encoder/Incremental/EC11/EC11E15204A3.html")
     (tags "rotary encoder")
@@
   )
   (footprint "MCU_RaspberryPi_and_Boards:RPi_Pico_SMD_TH" (layer "F.Cu")
-    (at 44.45 88.9)
+    (at 44.45 87.3125)
     (descr "Through hole straight pin header, 2x20, 2.54mm pitch, double rows")
     (tags "Through hole pin header THT 2x20 2.54mm double row")
@@
   )
   (footprint "Connector_PinSocket_2.54mm:PinSocket_1x14_P2.54mm_Vertical" (layer "F.Cu")
-    (at 27.80625 73.50125)
+    (at 29.36875 72.86625)
     (descr "Through hole straight socket strip, 1x14, 2.54mm pitch, single row (from Kicad 4.0.7), script generated")
     (tags "Through hole socket strip THT 1x14 2.54mm single row")
@@
     )
   )
-  (gr_line (start 286.54375 61.11875) (end 25.4 61.11875) (layer "Edge.Cuts") (width 0.1))
-  (gr_arc (start 25.4 137.31875) (mid 24.838749 137.086251) (end 24.60625 136.525) (layer "Edge.Cuts") (width 0.1))
-  (gr_arc (start 24.60625 61.9125) (mid 24.838731 61.351216) (end 25.4 61.11875) (layer "Edge.Cuts") (width 0.1))
-  (gr_line (start 24.60625 136.525) (end 24.60625 61.9125) (layer "Edge.Cuts") (width 0.1))
+  (gr_arc (start 27.78125 137.31875) (mid 27.220013 137.086237) (end 26.9875 136.525) (layer "Edge.Cuts") (width 0.1))
+  (gr_arc (start 26.9875 61.9125) (mid 27.219984 61.351234) (end 27.78125 61.11875) (layer "Edge.Cuts") (width 0.1))
+  (gr_line (start 27.78125 61.11875) (end 286.54375 61.11875) (layer "Edge.Cuts") (width 0.1))
+  (gr_line (start 26.9875 136.525) (end 26.9875 61.9125) (layer "Edge.Cuts") (width 0.1))
   (gr_line (start 287.3375 136.525) (end 287.3375 61.9125) (layer "Edge.Cuts") (width 0.1))
+  (gr_line (start 286.54375 137.31875) (end 27.78125 137.31875) (layer "Edge.Cuts") (width 0.1))
   (gr_arc (start 286.54375 61.11875) (mid 287.105016 61.351234) (end 287.3375 61.9125) (layer "Edge.Cuts") (width 0.1))
   (gr_arc (start 287.3375 136.525) (mid 287.104998 137.086234) (end 286.54375 137.31875) (layer "Edge.Cuts") (width 0.1))
-  (gr_line (start 286.54375 137.31875) (end 25.4 137.31875) (layer "Edge.Cuts") (width 0.1))
 )
